Commit message: Finished lab.

File: urdf/navvis.xacro (robot description, xacro)
@@ -1,4 +1,5 @@
 <?xml version="1.0"?>
 <robot xmlns:xacro="http://www.ros.org/wiki/xacro" name="navvis">
+  <xacro:include filename="$(find gazebo_plugins)/test/multi_robot_scenario/xacro/laser/hokuyo.xacro" />
   <link name="base">
     <visual>
@@ -15,72 +16,39 @@
     </collision>
   </link>
-  <link name="laser_vert_bottom">
-    <visual>
-      <geometry>
-        <box size="0.062 0.062 0.087" />
-      </geometry>
-    </visual>
-    <collision>
-      <geometry>
-        <box size="0.062 0.062 0.087" />
-      </geometry>
-    </collision>
-  </link>
-  <joint name="base_laser_vert_bottom_joint" type="fixed">
-    <parent link="base" />
-    <child link="laser_vert_bottom" />
-    <origin xyz="0.3158 -0.0021 0.5100" rpy="3.1355 -1.3045 0.0025" />
-  </joint>
-  <link name="laser_vert_top_right">
-    <visual>
-      <geometry>
-        <box size="0.062 0.062 0.087" />
-      </geometry>
-    </visual>
-    <collision>
-      <geometry>
-        <box size="0.062 0.062 0.087" />
-      </geometry>
-    </collision>
-  </link>
-  <joint name="base_laser_vert_top_right_joint" type="fixed">
-    <parent link="base" />
-    <child link="laser_vert_top_right" />
-    <origin xyz="0.2978 -0.1450 1.8451" rpy="-1.1760 0.6313 -1.9377" />
-  </joint>
-  <link name="laser_vert_top_left">
-    <visual>
-      <geometry>
-        <box size="0.062 0.062 0.087" />
-      </geometry>
-    </visual>
-    <collision>
-      <geometry>
-        <box size="0.062 0.062 0.087" />
-      </geometry>
-    </collision>
-  </link>
-  <joint name="base_laser_vert_top_left_joint" type="fixed">
-    <parent link="base" />
-    <child link="laser_vert_top_left" />
-    <origin xyz="0.2997 0.1531 1.8443" rpy=" 1.1780 0.6198 1.9560" />
-  </joint>
-  <link name="laser_horiz">
-    <visual>
-      <geometry>
-        <cylinder radius="0.052" length="0.072" />
-      </geometry>
-    </visual>
-    <collision>
-      <geometry>
-        <cylinder radius="0.052" length="0.072" />
-      </geometry>
-    </collision>
-  </link>
-  <joint name="base_laser_horiz_joint" type="fixed">
-    <parent link="base" />
-    <child link="laser_horiz" />
-    <origin xyz="0.2325 0.0001 1.9201" rpy="0.0012 0.1146 -0.0015" />
-  </joint>
+  <xacro:laser
+    name="laser_vert_bottom"
+    parent="base"
+    xyz="0.3158 -0.0021 0.5100"
+    rpy="3.1355 -1.3045 0.0025"
+    meshes="package://gazebo_plugins/test/multi_robot_scenario/meshes/laser"
+  />
+  <xacro:laser
+    name="laser_vert_top_right"
+    parent="base"
+    xyz="0.2978 -0.1450 1.8451"
+    rpy="-1.1760 0.6313 -1.9377"
+    meshes="package://gazebo_plugins/test/multi_robot_scenario/meshes/laser"
+  />
+  <xacro:laser
+    name="laser_vert_top_left"
+    parent="base"
+    xyz="0.2997 0.1531 1.8443"
+    rpy="1.1780 0.6198 1.9560"
+    meshes="package://gazebo_plugins/test/multi_robot_scenario/meshes/laser"
+  />
+  <xacro:include filename="$(find velodyne_description)/urdf/VLP-16.urdf.xacro"/>
+  <xacro:VLP-16
+    parent="base"
+    name="laser_horiz"
+    topic="laser_horiz/packets"
+    hz="10"
+    samples="440"
+    gpu="false"
+  >
+    <origin
+      xyz="0.2325416305773505 -0.0001380069427607134 1.920122926231907"
+      rpy="-0.0012068 0.114646 -0.0015308"
+    />
+  </xacro:VLP-16>
   <xacro:macro name="wheel_macro" params="side reflect">
     <link name="wheel_${side}">
@@ -125,4 +93,3 @@
     <axis xyz="0 0 1" />
   </joint>
-  <xacro:include filename="$(find gazebo_plugins)/test/multi_robot_scenario/xacro/laser/hokuyo.xacro" />
 </robot>
